File: electronics/board.brd (EAGLE design)
At the start: 130 x 54 mm, 9 parts

Commit message: small changes to initial board layout
Parts:
- added J10, J4: POWER_JACK, SparkFun-Connectors:POWER_JACK_PTH
- added U$2, U$3, U$4, U$5: M012MM-HOLE, abysscore:M01-2MM
- moved U$1 7.36 mm to (106.8, 11.8)
Connections:
- new net 12V: J4.PWR, U$3.P$1
- new net GND: J10.GND, J4.GND, U$5.P$1
- new net IN-: U$2.P$1
- new net OUT+1: U$4.P$1
- new net OUT+2: J10.PWR
Routing:
- net N$1: track 112.3 -> 106.4 mm
- net N$2: track 112.3 -> 107.1 mm
- net N$3: track 116.3 -> 112.1 mm
- net N$4: track 63.6 -> 60.2 mm
- net N$7: track 31.3 -> 34.0 mm
- net N$5: track 62.9 -> 60.2 mm
- net N$8: track 29.3 -> 32.0 mm
- net N$9: track 27.4 -> 30.0 mm
- net N$6: track 61.7 -> 59.7 mm
Changed lines of the file:
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@@
 </autorouter>
 <elements>
-<element name="U$1" library="abysscore" package="TSSOP24" value="AD5206" x="114.15" y="11.81" smashed="yes" rot="R270">
-<attribute name="NAME" x="112.0672" y="16.0056" size="1.016" layer="25" ratio="10"/>
-<attribute name="VALUE" x="112.0672" y="6.6238" size="1.016" layer="27" ratio="10"/>
+<element name="U$1" library="abysscore" package="TSSOP24" value="AD5206" x="106.79" y="11.81" smashed="yes" rot="R270">
+<attribute name="NAME" x="104.7072" y="16.0056" size="1.016" layer="25" ratio="10"/>
+<attribute name="VALUE" x="104.7072" y="6.6238" size="1.016" layer="27" ratio="10"/>
 </element>
 <element name="J1" library="SparkFun-Connectors" library_urn="urn:adsk.eagle:library:513" package="1X03" package3d_urn="urn:adsk.eagle:package:38063/1" value="" x="20.8" y="2.54" smashed="yes" rot="R90">
@@
 <attribute name="VALUE" x="62.23" y="3.197" size="0.6096" layer="27" font="vector" ratio="20" rot="R180"/>
 </element>
+<element name="U$2" library="abysscore" package="M01-2MM" value="M012MM-HOLE" x="4.03" y="21.52" smashed="yes"/>
+<element name="U$3" library="abysscore" package="M01-2MM" value="M012MM-HOLE" x="3.75" y="28.18" smashed="yes"/>
+<element name="U$4" library="abysscore" package="M01-2MM" value="M012MM-HOLE" x="123.67" y="30.17" smashed="yes"/>
+<element name="U$5" library="abysscore" package="M01-2MM" value="M012MM-HOLE" x="123.75" y="23.2" smashed="yes"/>
+<element name="J4" library="SparkFun-Connectors" library_urn="urn:adsk.eagle:library:513" package="POWER_JACK_PTH" package3d_urn="urn:adsk.eagle:package:38231/1" value="POWER_JACK" x="-3.06" y="14.37" smashed="yes" rot="R270">
+<attribute name="NAME" x="-1.2312" y="15.7416" size="0.6096" layer="25" font="vector" ratio="20" rot="R270"/>
+<attribute name="PROD_ID" value="CONN-08197" x="-3.06" y="14.37" size="1.778" layer="27" rot="R270" display="off"/>
+<attribute name="VALUE" x="-2.2472" y="16.1226" size="0.6096" layer="27" font="vector" ratio="20" rot="R270"/>
+</element>
+<element name="J10" library="SparkFun-Connectors" library_urn="urn:adsk.eagle:library:513" package="POWER_JACK_PTH" package3d_urn="urn:adsk.eagle:package:38231/1" value="POWER_JACK" x="134.27" y="12.17" smashed="yes" rot="R90">
+<attribute name="NAME" x="132.4412" y="10.7984" size="0.6096" layer="25" font="vector" ratio="20" rot="R90"/>
+<attribute name="PROD_ID" value="CONN-08197" x="134.27" y="12.17" size="1.778" layer="27" rot="R90" display="off"/>
+<attribute name="VALUE" x="133.4572" y="10.4174" size="0.6096" layer="27" font="vector" ratio="20" rot="R90"/>
+</element>
 </elements>
 <signals>
@@
 <wire x1="60.36" y1="10.53" x2="70.48" y2="10.53" width="0.25" layer="1"/>
 <wire x1="70.48" y1="10.53" x2="70.48" y2="5.66" width="0.25" layer="1"/>
-<wire x1="70.48" y1="5.66" x2="117.9104" y2="5.6272" width="0.25" layer="1"/>
-<wire x1="117.9104" y1="8.235" x2="117.0678" y2="8.235" width="0.25" layer="1"/>
-<wire x1="117.9104" y1="5.6272" x2="117.9104" y2="8.235" width="0.25" layer="1"/>
+<wire x1="70.48" y1="5.66" x2="111.2804" y2="5.631784375" width="0.25" layer="1"/>
+<wire x1="111.2804" y1="8.235" x2="109.7078" y2="8.235" width="0.25" layer="1"/>
+<wire x1="111.2804" y1="5.631784375" x2="111.2804" y2="8.235" width="0.25" layer="1"/>
 </signal>
 <signal name="N$2">
@@
 <contactref element="J1" pad="2"/>
 <wire x1="20.8" y1="5.08" x2="20.9448" y2="5.2248" width="0.25" layer="1"/>
-<wire x1="118.3228" y1="5.2248" x2="69.97" y2="5.2248" width="0.25" layer="1"/>
+<wire x1="112.0828" y1="5.2248" x2="69.97" y2="5.2248" width="0.25" layer="1"/>
 <wire x1="69.97" y1="5.2248" x2="69.97" y2="10.11" width="0.25" layer="1"/>
 <wire x1="69.97" y1="10.11" x2="60.8" y2="10.11" width="0.25" layer="1"/>
 <wire x1="60.8" y1="10.11" x2="60.8" y2="5.2248" width="0.25" layer="1"/>
 <wire x1="60.8" y1="5.2248" x2="20.9448" y2="5.2248" width="0.25" layer="1"/>
-<wire x1="118.3228" y1="8.885" x2="117.0678" y2="8.885" width="0.25" layer="1"/>
-<wire x1="118.3228" y1="5.2248" x2="118.3228" y2="8.885" width="0.25" layer="1"/>
+<wire x1="112.0828" y1="8.885" x2="109.7078" y2="8.885" width="0.25" layer="1"/>
+<wire x1="112.0828" y1="5.2248" x2="112.0828" y2="8.885" width="0.25" layer="1"/>
 </signal>
 <signal name="N$3">
@@
 <wire x1="61.26" y1="9.69" x2="69.47" y2="9.69" width="0.25" layer="1"/>
 <wire x1="69.47" y1="9.69" x2="69.47" y2="4.8224" width="0.25" layer="1"/>
-<wire x1="69.47" y1="4.8224" x2="118.7252" y2="4.8224" width="0.25" layer="1"/>
-<wire x1="118.7252" y1="9.535" x2="117.0678" y2="9.535" width="0.25" layer="1"/>
-<wire x1="118.7252" y1="4.8224" x2="118.7252" y2="9.535" width="0.25" layer="1"/>
+<wire x1="69.47" y1="4.8224" x2="112.9452" y2="4.8224" width="0.25" layer="1"/>
+<wire x1="112.9452" y1="9.535" x2="109.7078" y2="9.535" width="0.25" layer="1"/>
+<wire x1="112.9452" y1="4.8224" x2="112.9452" y2="9.535" width="0.25" layer="1"/>
 </signal>
 <signal name="N$4">
@@
 <wire x1="67.86" y1="3.83" x2="66.4" y2="3.83" width="0.25" layer="1"/>
 <wire x1="66.4" y1="3.83" x2="65.11" y2="2.54" width="0.25" layer="1"/>
-<wire x1="67.86" y1="4.4" x2="119.1476" y2="4.4" width="0.25" layer="1"/>
-<wire x1="119.1476" y1="4.4" x2="119.1476" y2="10.185" width="0.25" layer="1"/>
-<wire x1="119.1476" y1="10.185" x2="117.0678" y2="10.185" width="0.25" layer="1"/>
+<wire x1="67.86" y1="4.4" x2="113.7576" y2="4.4" width="0.25" layer="1"/>
+<wire x1="113.7576" y1="4.4" x2="113.7576" y2="10.185" width="0.25" layer="1"/>
+<wire x1="113.7576" y1="10.185" x2="109.7078" y2="10.185" width="0.25" layer="1"/>
 </signal>
 <signal name="N$5">
@@
 <wire x1="68.44" y1="3.19" x2="67.69" y2="3.19" width="0.25" layer="1"/>
 <wire x1="68.44" y1="3.19" x2="68.44" y2="3.98" width="0.25" layer="1"/>
-<wire x1="68.44" y1="3.98" x2="119.57" y2="3.98" width="0.25" layer="1"/>
-<wire x1="119.57" y1="3.98" x2="119.57" y2="10.835" width="0.25" layer="1"/>
-<wire x1="119.57" y1="10.835" x2="117.0678" y2="10.835" width="0.25" layer="1"/>
+<wire x1="68.44" y1="3.98" x2="114.51" y2="3.98" width="0.25" layer="1"/>
+<wire x1="114.51" y1="3.98" x2="114.51" y2="10.835" width="0.25" layer="1"/>
+<wire x1="114.51" y1="10.835" x2="109.7078" y2="10.835" width="0.25" layer="1"/>
 </signal>
 <signal name="N$6">
@@
 <contactref element="J2" pad="1"/>
 <wire x1="69.58" y1="2.54" x2="70.6" y2="3.56" width="0.25" layer="1"/>
-<wire x1="120" y1="3.56" x2="70.6" y2="3.56" width="0.25" layer="1"/>
-<wire x1="120" y1="11.485" x2="117.0678" y2="11.485" width="0.25" layer="1"/>
-<wire x1="120" y1="3.56" x2="120" y2="11.485" width="0.25" layer="1"/>
+<wire x1="115.33" y1="3.56" x2="70.6" y2="3.56" width="0.25" layer="1"/>
+<wire x1="115.33" y1="11.485" x2="109.7078" y2="11.485" width="0.25" layer="1"/>
+<wire x1="115.33" y1="3.56" x2="115.33" y2="11.485" width="0.25" layer="1"/>
 </signal>
 <signal name="N$7">
 <contactref element="U$1" pad="19"/>
 <contactref element="J3" pad="3"/>
-<wire x1="124.35" y1="38.6" x2="120.11" y2="34.36" width="0.25" layer="1"/>
-<wire x1="120.11" y1="34.36" x2="120.11" y2="12.135" width="0.25" layer="1"/>
-<wire x1="120.11" y1="12.135" x2="117.0678" y2="12.135" width="0.25" layer="1"/>
+<wire x1="124.35" y1="38.6" x2="112.29" y2="26.54" width="0.25" layer="1"/>
+<wire x1="112.29" y1="26.54" x2="112.29" y2="12.135" width="0.25" layer="1"/>
+<wire x1="112.29" y1="12.135" x2="109.7078" y2="12.135" width="0.25" layer="1"/>
 </signal>
 <signal name="N$8">
 <contactref element="U$1" pad="20"/>
 <contactref element="J3" pad="2"/>
-<wire x1="121.81" y1="38.6" x2="119.69" y2="36.48" width="0.25" layer="1"/>
-<wire x1="119.69" y1="36.48" x2="119.69" y2="12.785" width="0.25" layer="1"/>
-<wire x1="119.69" y1="12.785" x2="117.0678" y2="12.785" width="0.25" layer="1"/>
+<wire x1="121.81" y1="38.6" x2="111.65" y2="28.44" width="0.25" layer="1"/>
+<wire x1="111.65" y1="28.44" x2="111.65" y2="12.785" width="0.25" layer="1"/>
+<wire x1="111.65" y1="12.785" x2="109.7078" y2="12.785" width="0.25" layer="1"/>
 </signal>
 <signal name="N$9">
 <contactref element="U$1" pad="21"/>
 <contactref element="J3" pad="1"/>
-<wire x1="119.27" y1="38.6" x2="119.27" y2="13.435" width="0.25" layer="1"/>
-<wire x1="119.27" y1="13.435" x2="117.0678" y2="13.435" width="0.25" layer="1"/>
+<wire x1="119.27" y1="38.6" x2="111.12" y2="30.45" width="0.25" layer="1"/>
+<wire x1="111.12" y1="30.45" x2="111.12" y2="13.435" width="0.25" layer="1"/>
+<wire x1="111.12" y1="13.435" x2="109.7078" y2="13.435" width="0.25" layer="1"/>
 </signal>
 <signal name="N$10">
@@
 <contactref element="U$1" pad="9"/>
 </signal>
+<signal name="IN-">
+<contactref element="U$2" pad="P$1"/>
+</signal>
+<signal name="GND">
+<contactref element="J4" pad="GND"/>
+<contactref element="U$5" pad="P$1"/>
+<contactref element="J10" pad="GND"/>
+<wire x1="4.64" y1="14.37" x2="126.57" y2="12.17" width="0" layer="19" extent="1-1"/>
+<wire x1="123.75" y1="23.2" x2="4.64" y2="14.37" width="0" layer="19" extent="1-1"/>
+</signal>
+<signal name="12V">
+<contactref element="J4" pad="PWR"/>
+<contactref element="U$3" pad="P$1"/>
+<wire x1="3.75" y1="28.18" x2="10.64" y2="14.37" width="0" layer="19" extent="1-1"/>
+</signal>
+<signal name="OUT+1">
+<contactref element="U$4" pad="P$1"/>
+</signal>
+<signal name="OUT+2">
+<contactref element="J10" pad="PWR"/>
+</signal>
 </signals>

Commit message: small changes to initial board layout
Parts:
- moved J10 1.20 mm to (133.1, 12.2)
Connections:
- removed net N$10: U$1.6
- removed net N$11: U$1.4
- removed net N$12: U$1.5
- removed net N$13: U$1.8
- removed net N$14: U$1.7
- removed net N$15: U$1.9
- new net 3.3V: J5.5
- new net 5V: J5.4, U$1.6
- new net A0: J8.5
- new net A1: J8.4
- new net A2: J8.3
- new net A3: J8.2
- new net A4: J8.1
- new net D0: J6.1
- new net D1: J6.2
- new net D2: J6.3
- new net D3: J6.4
- new net D4: J6.5
- new net D5: J6.6
- new net D6: J6.7
- new net D7: J6.8
- new net D8: J7.1
- new net D9: J7.2
- new net MISO: J7.5
- new net MOSI: J7.4, U$1.7
- new net SCK: J7.6, U$1.8
- new net SS: J7.3, U$1.5
- net 12V: now also J5.1
- net GND: now also J5.2, J5.3, U$1.4, U$1.9
Routing:
- net N$1: track 106.4 -> 95.2 mm
- net N$3: track 112.1 -> 101.0 mm
- net N$2: track 107.1 -> 97.3 mm
