File: electronics/board.sch (EAGLE design)
At the start: 9 parts

Commit message: small changes to initial board layout
Parts:
- added J10, J4: POWER_JACK, SparkFun-Connectors:POWER_JACK
- added U$2, U$3, U$4, U$5: M012MM-HOLE, abysscore:M012MM-HOLE
Connections:
- new net 12V: J4.PWR, U$3.P$1
- new net GND: J10.GND, J4.GND, U$5.P$1
- new net IN-: U$2.P$1
- new net OUT+1: U$4.P$1
- new net OUT+2: J10.PWR
Changed lines of the file:
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@@
 <part name="J5" library="SparkFun-Connectors" library_urn="urn:adsk.eagle:library:513" deviceset="CONN_08" device="&quot;" package3d_urn="urn:adsk.eagle:package:38138/1"/>
 <part name="J8" library="SparkFun-Connectors" library_urn="urn:adsk.eagle:library:513" deviceset="CONN_05" device="" package3d_urn="urn:adsk.eagle:package:38104/1"/>
+<part name="U$2" library="abysscore" deviceset="M01" device="2MM-HOLE"/>
+<part name="U$3" library="abysscore" deviceset="M01" device="2MM-HOLE"/>
+<part name="U$4" library="abysscore" deviceset="M01" device="2MM-HOLE"/>
+<part name="U$5" library="abysscore" deviceset="M01" device="2MM-HOLE"/>
+<part name="J4" library="SparkFun-Connectors" library_urn="urn:adsk.eagle:library:513" deviceset="POWER_JACK" device="" package3d_urn="urn:adsk.eagle:package:38231/1"/>
+<part name="J10" library="SparkFun-Connectors" library_urn="urn:adsk.eagle:library:513" deviceset="POWER_JACK" device="" package3d_urn="urn:adsk.eagle:package:38231/1"/>
 </parts>
 <sheets>
@@
 <attribute name="NAME" x="-25.4" y="102.108" size="1.778" layer="95" font="vector"/>
 </instance>
+<instance part="U$2" gate="G$1" x="-96.52" y="55.88" smashed="yes" rot="R180"/>
+<instance part="U$3" gate="G$1" x="-96.52" y="48.26" smashed="yes" rot="R180"/>
+<instance part="U$4" gate="G$1" x="167.64" y="66.04" smashed="yes"/>
+<instance part="U$5" gate="G$1" x="167.64" y="58.42" smashed="yes"/>
+<instance part="J4" gate="G$1" x="-91.44" y="30.48" smashed="yes">
+<attribute name="VALUE" x="-101.6" y="40.64" size="1.778" layer="96" font="vector"/>
+<attribute name="NAME" x="-101.6" y="30.48" size="1.778" layer="95" font="vector"/>
+</instance>
+<instance part="J10" gate="G$1" x="165.1" y="33.02" smashed="yes" rot="R180">
+<attribute name="VALUE" x="175.26" y="22.86" size="1.778" layer="96" font="vector" rot="R180"/>
+<attribute name="NAME" x="175.26" y="33.02" size="1.778" layer="95" font="vector" rot="R180"/>
+</instance>
 </instances>
 <busses>
@@
 </segment>
 </net>
+<net name="IN-" class="0">
+<segment>
+<pinref part="U$2" gate="G$1" pin="P$1"/>
+<wire x1="-88.9" y1="55.88" x2="-73.66" y2="55.88" width="0.1524" layer="91"/>
+<label x="-81.28" y="55.88" size="1.778" layer="95"/>
+</segment>
+</net>
+<net name="GND" class="0">
+<segment>
+<pinref part="J4" gate="G$1" pin="GND"/>
+<wire x1="-88.9" y1="33.02" x2="-81.28" y2="33.02" width="0.1524" layer="91"/>
+<label x="-86.36" y="33.02" size="1.778" layer="95"/>
+</segment>
+<segment>
+<pinref part="U$5" gate="G$1" pin="P$1"/>
+<wire x1="160.02" y1="58.42" x2="152.4" y2="58.42" width="0.1524" layer="91"/>
+<label x="152.4" y="58.42" size="1.778" layer="95"/>
+</segment>
+<segment>
+<pinref part="J10" gate="G$1" pin="GND"/>
+<wire x1="162.56" y1="30.48" x2="152.4" y2="30.48" width="0.1524" layer="91"/>
+<label x="152.4" y="30.48" size="1.778" layer="95"/>
+</segment>
+</net>
+<net name="12V" class="0">
+<segment>
+<pinref part="J4" gate="G$1" pin="PWR"/>
+<wire x1="-88.9" y1="38.1" x2="-81.28" y2="38.1" width="0.1524" layer="91"/>
+<label x="-86.36" y="38.1" size="1.778" layer="95"/>
+</segment>
+<segment>
+<pinref part="U$3" gate="G$1" pin="P$1"/>
+<wire x1="-88.9" y1="48.26" x2="-73.66" y2="48.26" width="0.1524" layer="91"/>
+<label x="-81.28" y="48.26" size="1.778" layer="95"/>
+</segment>
+</net>
+<net name="OUT+1" class="0">
+<segment>
+<pinref part="U$4" gate="G$1" pin="P$1"/>
+<wire x1="160.02" y1="66.04" x2="152.4" y2="66.04" width="0.1524" layer="91"/>
+<label x="152.4" y="66.04" size="1.778" layer="95"/>
+</segment>
+</net>
+<net name="OUT+2" class="0">
+<segment>
+<pinref part="J10" gate="G$1" pin="PWR"/>
+<wire x1="162.56" y1="25.4" x2="152.4" y2="25.4" width="0.1524" layer="91"/>
+<label x="152.4" y="25.4" size="1.778" layer="95"/>
+</segment>
+</net>

Commit message: small changes to initial board layout
Connections:
- removed net N$10: U$1.VDD
- removed net N$11: U$1.GND
- removed net N$12: U$1.CS
- removed net N$13: U$1.CLK
- removed net N$14: U$1.SDI
- removed net N$15: U$1.VSS
- new net 3.3V: J5.5
- new net 5V: J5.4, U$1.VDD
- new net A0: J8.5
- new net A1: J8.4
- new net A2: J8.3
- new net A3: J8.2
- new net A4: J8.1
- new net D0: J6.1
- new net D1: J6.2
- new net D2: J6.3
- new net D3: J6.4
- new net D4: J6.5
- new net D5: J6.6
- new net D6: J6.7
- new net D7: J6.8
- new net D8: J7.1
- new net D9: J7.2
- new net MISO: J7.5
- new net MOSI: J7.4, U$1.SDI
- new net SCK: J7.6, U$1.CLK
- new net SS: J7.3, U$1.CS
- net 12V: now also J5.1
- net GND: now also J5.2, J5.3, U$1.GND, U$1.VSS
Other:
- moved on the sheet: J8
Changed lines of the file:
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@@
 <attribute name="NAME" x="-7.62" y="79.248" size="1.778" layer="95" font="vector"/>
 </instance>
-<instance part="J8" gate="G$1" x="-22.86" y="93.98" smashed="yes">
-<attribute name="VALUE" x="-25.4" y="84.074" size="1.778" layer="96" font="vector"/>
-<attribute name="NAME" x="-25.4" y="102.108" size="1.778" layer="95" font="vector"/>
+<instance part="J8" gate="G$1" x="-5.08" y="93.98" smashed="yes">
+<attribute name="VALUE" x="-7.62" y="84.074" size="1.778" layer="96" font="vector"/>
+<attribute name="NAME" x="-7.62" y="102.108" size="1.778" layer="95" font="vector"/>
 </instance>
 <instance part="U$2" gate="G$1" x="-96.52" y="55.88" smashed="yes" rot="R180"/>
@@
 </segment>
 </net>
-<net name="N$10" class="0">
-<segment>
-<pinref part="U$1" gate="G$1" pin="VDD"/>
-<wire x1="60.96" y1="50.8" x2="33.02" y2="50.8" width="0.1524" layer="91"/>
-</segment>
-</net>
-<net name="N$11" class="0">
-<segment>
-<pinref part="U$1" gate="G$1" pin="GND"/>
-<wire x1="60.96" y1="55.88" x2="33.02" y2="55.88" width="0.1524" layer="91"/>
-</segment>
-</net>
-<net name="N$12" class="0">
-<segment>
-<pinref part="U$1" gate="G$1" pin="CS"/>
-<wire x1="60.96" y1="53.34" x2="33.02" y2="53.34" width="0.1524" layer="91"/>
-</segment>
-</net>
-<net name="N$13" class="0">
-<segment>
-<pinref part="U$1" gate="G$1" pin="CLK"/>
-<wire x1="60.96" y1="45.72" x2="33.02" y2="45.72" width="0.1524" layer="91"/>
-</segment>
-</net>
-<net name="N$14" class="0">
-<segment>
-<pinref part="U$1" gate="G$1" pin="SDI"/>
-<wire x1="60.96" y1="48.26" x2="33.02" y2="48.26" width="0.1524" layer="91"/>
-</segment>
-</net>
-<net name="N$15" class="0">
-<segment>
-<pinref part="U$1" gate="G$1" pin="VSS"/>
-<wire x1="60.96" y1="43.18" x2="33.02" y2="43.18" width="0.1524" layer="91"/>
-</segment>
-</net>
 <net name="IN-" class="0">
 <segment>
@@
 <label x="152.4" y="30.48" size="1.778" layer="95"/>
 </segment>
+<segment>
+<pinref part="J5" gate="G$1" pin="3"/>
+<wire x1="2.54" y1="63.5" x2="12.7" y2="63.5" width="0.1524" layer="91"/>
+<label x="7.62" y="63.5" size="1.778" layer="95"/>
+</segment>
+<segment>
+<pinref part="J5" gate="G$1" pin="2"/>
+<wire x1="2.54" y1="60.96" x2="12.7" y2="60.96" width="0.1524" layer="91"/>
+<label x="7.62" y="60.96" size="1.778" layer="95"/>
+</segment>
+<segment>
+<pinref part="U$1" gate="G$1" pin="GND"/>
+<wire x1="60.96" y1="55.88" x2="33.02" y2="55.88" width="0.1524" layer="91"/>
+<label x="33.02" y="55.88" size="1.778" layer="95"/>
+</segment>
+<segment>
+<pinref part="U$1" gate="G$1" pin="VSS"/>
+<wire x1="60.96" y1="43.18" x2="33.02" y2="43.18" width="0.1524" layer="91"/>
+<label x="33.02" y="43.18" size="1.778" layer="95"/>
+</segment>
 </net>
 <net name="12V" class="0">
@@
 <label x="-81.28" y="48.26" size="1.778" layer="95"/>
 </segment>
+<segment>
+<pinref part="J5" gate="G$1" pin="1"/>
+<wire x1="2.54" y1="58.42" x2="12.7" y2="58.42" width="0.1524" layer="91"/>
+<label x="7.62" y="58.42" size="1.778" layer="95"/>
+</segment>
 </net>
 <net name="OUT+1" class="0">
@@
 </segment>
 </net>
+<net name="5V" class="0">
+<segment>
+<pinref part="J5" gate="G$1" pin="4"/>
+<wire x1="2.54" y1="66.04" x2="12.7" y2="66.04" width="0.1524" layer="91"/>
+<label x="7.62" y="66.04" size="1.778" layer="95"/>
+</segment>
+<segment>
+<pinref part="U$1" gate="G$1" pin="VDD"/>
+<wire x1="60.96" y1="50.8" x2="33.02" y2="50.8" width="0.1524" layer="91"/>
+<label x="33.02" y="50.8" size="1.778" layer="95"/>
+</segment>
+</net>
+<net name="3.3V" class="0">
+<segment>
+<pinref part="J5" gate="G$1" pin="5"/>
+<wire x1="2.54" y1="68.58" x2="12.7" y2="68.58" width="0.1524" layer="91"/>
+<label x="7.62" y="68.58" size="1.778" layer="95"/>
+</segment>
+</net>
+<net name="A0" class="0">
+<segment>
+<pinref part="J8" gate="G$1" pin="5"/>
+<wire x1="2.54" y1="99.06" x2="15.24" y2="99.06" width="0.1524" layer="91"/>
+<label x="12.7" y="99.06" size="1.778" layer="95"/>
+</segment>
+</net>
+<net name="A1" class="0">
+<segment>
+<pinref part="J8" gate="G$1" pin="4"/>
+<wire x1="2.54" y1="96.52" x2="15.24" y2="96.52" width="0.1524" layer="91"/>
+<label x="12.7" y="96.52" size="1.778" layer="95"/>
+</segment>
+</net>
+<net name="A2" class="0">
+<segment>
+<pinref part="J8" gate="G$1" pin="3"/>
+<wire x1="2.54" y1="93.98" x2="15.24" y2="93.98" width="0.1524" layer="91"/>
+<label x="12.7" y="93.98" size="1.778" layer="95"/>
+</segment>
+</net>
+<net name="A3" class="0">
+<segment>
+<pinref part="J8" gate="G$1" pin="2"/>
+<wire x1="2.54" y1="91.44" x2="15.24" y2="91.44" width="0.1524" layer="91"/>
+<label x="12.7" y="91.44" size="1.778" layer="95"/>
+</segment>
+</net>
+<net name="A4" class="0">
+<segment>
+<pinref part="J8" gate="G$1" pin="1"/>
+<wire x1="2.54" y1="88.9" x2="15.24" y2="88.9" width="0.1524" layer="91"/>
+<label x="12.7" y="88.9" size="1.778" layer="95"/>
+</segment>
+</net>
+<net name="SCK" class="0">
+<segment>
+<pinref part="J7" gate="G$1" pin="6"/>
+<wire x1="5.08" y1="15.24" x2="15.24" y2="15.24" width="0.1524" layer="91"/>
+<label x="10.16" y="15.24" size="1.778" layer="95"/>
+</segment>
+<segment>
+<pinref part="U$1" gate="G$1" pin="CLK"/>
+<wire x1="60.96" y1="45.72" x2="33.02" y2="45.72" width="0.1524" layer="91"/>
+<label x="33.02" y="45.72" size="1.778" layer="95"/>
+</segment>
+</net>
+<net name="MISO" class="0">
+<segment>
+<pinref part="J7" gate="G$1" pin="5"/>
+<wire x1="5.08" y1="12.7" x2="15.24" y2="12.7" width="0.1524" layer="91"/>
+<label x="10.16" y="12.7" size="1.778" layer="95"/>
+</segment>
+</net>
+<net name="MOSI" class="0">
+<segment>
+<pinref part="J7" gate="G$1" pin="4"/>
+<wire x1="5.08" y1="10.16" x2="15.24" y2="10.16" width="0.1524" layer="91"/>
+<label x="10.16" y="10.16" size="1.778" layer="95"/>
+</segment>
+<segment>
+<pinref part="U$1" gate="G$1" pin="SDI"/>
+<wire x1="60.96" y1="48.26" x2="33.02" y2="48.26" width="0.1524" layer="91"/>
+<label x="33.02" y="48.26" size="1.778" layer="95"/>
+</segment>
+</net>
+<net name="SS" class="0">
+<segment>
+<pinref part="J7" gate="G$1" pin="3"/>
+<wire x1="5.08" y1="7.62" x2="15.24" y2="7.62" width="0.1524" layer="91"/>
+<label x="10.16" y="7.62" size="1.778" layer="95"/>
+</segment>
+<segment>
+<pinref part="U$1" gate="G$1" pin="CS"/>
+<wire x1="60.96" y1="53.34" x2="33.02" y2="53.34" width="0.1524" layer="91"/>
+<label x="33.02" y="53.34" size="1.778" layer="95"/>
+</segment>
+</net>
+<net name="D9" class="0">
+<segment>
+<pinref part="J7" gate="G$1" pin="2"/>
+<wire x1="5.08" y1="5.08" x2="15.24" y2="5.08" width="0.1524" layer="91"/>
+<label x="10.16" y="5.08" size="1.778" layer="95"/>
+</segment>
+</net>
+<net name="D8" class="0">
+<segment>
+<pinref part="J7" gate="G$1" pin="1"/>
+<wire x1="5.08" y1="2.54" x2="15.24" y2="2.54" width="0.1524" layer="91"/>
+<label x="10.16" y="2.54" size="1.778" layer="95"/>
+</segment>
+</net>
+<net name="D7" class="0">
+<segment>
+<pinref part="J6" gate="G$1" pin="8"/>
+<wire x1="5.08" y1="45.72" x2="12.7" y2="45.72" width="0.1524" layer="91"/>
+<label x="10.16" y="45.72" size="1.778" layer="95"/>
+</segment>
+</net>
+<net name="D6" class="0">
+<segment>
+<pinref part="J6" gate="G$1" pin="7"/>
+<wire x1="5.08" y1="43.18" x2="12.7" y2="43.18" width="0.1524" layer="91"/>
+<label x="10.16" y="43.18" size="1.778" layer="95"/>
+</segment>
+</net>
+<net name="D5" class="0">
+<segment>
+<pinref part="J6" gate="G$1" pin="6"/>
+<wire x1="5.08" y1="40.64" x2="12.7" y2="40.64" width="0.1524" layer="91"/>
+<label x="10.16" y="40.64" size="1.778" layer="95"/>
+</segment>
+</net>
+<net name="D4" class="0">
+<segment>
+<pinref part="J6" gate="G$1" pin="5"/>
+<wire x1="5.08" y1="38.1" x2="12.7" y2="38.1" width="0.1524" layer="91"/>
+<label x="10.16" y="38.1" size="1.778" layer="95"/>
+</segment>
+</net>
+<net name="D3" class="0">
+<segment>
+<pinref part="J6" gate="G$1" pin="4"/>
+<wire x1="5.08" y1="35.56" x2="12.7" y2="35.56" width="0.1524" layer="91"/>
+<label x="10.16" y="35.56" size="1.778" layer="95"/>
+</segment>
+</net>
+<net name="D2" class="0">
+<segment>
+<pinref part="J6" gate="G$1" pin="3"/>
+<wire x1="5.08" y1="33.02" x2="12.7" y2="33.02" width="0.1524" layer="91"/>
+<label x="10.16" y="33.02" size="1.778" layer="95"/>
+</segment>
+</net>
+<net name="D1" class="0">
+<segment>
+<pinref part="J6" gate="G$1" pin="2"/>
+<wire x1="5.08" y1="30.48" x2="12.7" y2="30.48" width="0.1524" layer="91"/>
+<label x="10.16" y="30.48" size="1.778" layer="95"/>
+</segment>
+</net>
+<net name="D0" class="0">
+<segment>
+<pinref part="J6" gate="G$1" pin="1"/>
+<wire x1="5.08" y1="27.94" x2="12.7" y2="27.94" width="0.1524" layer="91"/>
+<label x="10.16" y="27.94" size="1.778" layer="95"/>
+</segment>
+</net>
